File: kicad/beverageWarmer1.kicad_pcb (KiCad board)
At the start: 4 copper layers, 99.6 x 131.1 mm, 64 parts, among them J0 Conn_01x02, J1 Conn_01x02, U0 IRF7205TRPBF, U1 AD820ARMZ, U2 AD820ARMZ, U3 Op07DRZ, U4 Op07DRZ, U5 ADP1720, U6 TL750L10CD

Commit message: Final Sch Push?
Parts:
- removed C0: 22u, Capacitor_SMD:C_1210_3225Metric_Pad1.33x2.70mm_HandSolder
- removed C100: 10n, Capacitor_SMD:C_0603_1608Metric_Pad1.08x0.95mm_HandSolder
- removed C500, C501, C600, C601: 1u, Capacitor_SMD:C_0603_1608Metric_Pad1.08x0.95mm_HandSolder
- removed D0: DIODE, Diode_SMD:D_SMC
- removed D400: D_Zener, Diode_SMD:D_SMC
- removed J0: Conn_01x02, Connector_PinHeader_2.54mm:PinHeader_1x02_P2.54mm_Vertical_SMD_Pin1Right
- removed L0: 22u, customFootprints:MPXV1D1054
- removed R100, R101, R102, R103, R200, R300, R301, R302, R303, R305, R400: 1k, Resistor_SMD:R_0603_1608Metric_Pad0.98x0.95mm_HandSolder
- removed R201, R402: 10k, Resistor_SMD:R_0603_1608Metric_Pad0.98x0.95mm_HandSolder
- removed R304: 5.5k, Resistor_SMD:R_0603_1608Metric_Pad0.98x0.95mm_HandSolder
- removed R401, R404: 2k, Resistor_SMD:R_0603_1608Metric_Pad0.98x0.95mm_HandSolder
- removed R405: 0, Resistor_SMD:R_0603_1608Metric_Pad0.98x0.95mm_HandSolder
- removed TH401: Thermistor, Resistor_THT:R_Axial_DIN0204_L3.6mm_D1.6mm_P2.54mm_Vertical
- removed TP0, TP100, TP300, TP400, TP401, TP402: TestPoint, TestPoint:TestPoint_Pad_D2.5mm
- removed U0: IRF7205TRPBF, Package_SO:SOIC-8_3.9x4.9mm_P1.27mm
- added C10: 0.1u, Capacitor_SMD:C_0603_1608Metric, F.Cu at (260.0, 64.8)
- added C11: 0.1u, Capacitor_SMD:C_0603_1608Metric, F.Cu at (259.0, 74.9)
- added C12: 0.1u, Capacitor_SMD:C_0603_1608Metric, F.Cu at (247.0, 73.7)
- added C13: 0.1u, Capacitor_SMD:C_0603_1608Metric, F.Cu at (271.0, 51.0)
- added C14: 0.1u, Capacitor_SMD:C_0603_1608Metric, F.Cu at (250.7, 70.3)
- added C15: 1u, Capacitor_SMD:C_0603_1608Metric, F.Cu at (251.6, 80.7)
- added C16: 1u, Capacitor_SMD:C_0603_1608Metric, F.Cu at (263.1, 73.1)
- added C17: 0.1u, Capacitor_SMD:C_0603_1608Metric, F.Cu at (255.6, 80.7)
- added C18: 0.1u, Capacitor_SMD:C_0603_1608Metric, F.Cu at (272.0, 64.0)
- added C19: 1u, Capacitor_SMD:C_0603_1608Metric, F.Cu at (255.6, 78.2)
- added C2: 0.1u, Capacitor_SMD:C_0603_1608Metric, F.Cu at (264.0, 63.0)
- added C20: 0.1u, Capacitor_SMD:C_0603_1608Metric, F.Cu at (272.0, 61.5)
- added C3: 0.1u, Capacitor_SMD:C_0603_1608Metric, F.Cu at (251.0, 75.3)
- added C4: 10u, Capacitor_SMD:C_1206_3216Metric, F.Cu at (242.2, 75.1)
- added C5: 1u, Capacitor_SMD:C_0603_1608Metric, F.Cu at (267.6, 59.5)
- added C6: 1u, Capacitor_SMD:C_0603_1608Metric, F.Cu at (260.0, 67.3)
- added C7: 1u, Capacitor_SMD:C_0603_1608Metric, F.Cu at (270.8, 53.5)
- added C8: 1u, Capacitor_SMD:C_0603_1608Metric, F.Cu at (247.0, 76.2)
- added C9: 1u, Capacitor_SMD:C_0603_1608Metric, F.Cu at (251.0, 72.8)
- added D1: V3FL45, Diode_SMD:D_SMF, F.Cu at (245.9, 70.7)
- added D2: 5.6V, Diode_SMD:D_SOD-123, F.Cu at (228.1, 85.1)
- added D3: RED, LED_SMD:LED_0603_1608Metric, F.Cu at (235.6, 80.8)
- added D4: GREEN, LED_SMD:LED_0603_1608Metric, F.Cu at (241.4, 78.1)
- added D5: V3FL45, Diode_SMD:D_SMF, F.Cu at (233.8, 85.1)
- added D6: V3FL45, Diode_SMD:D_SMF, F.Cu at (255.1, 65.2)
- added F1: 3A, Fuse:Fuse_0603_1608Metric, F.Cu at (243.6, 80.6)
- added FB1: FB, Inductor_SMD:L_0603_1608Metric, F.Cu at (239.6, 83.2)
- added J2: CAN_CONN, Connector_Molex:Molex_Micro-Fit_3.0_43650-0200_1x02_P3.00mm_Horizontal, F.Cu at (244.9, 55.1)
- added J3: SWD, Connector_PinSocket_1.27mm:PinSocket_2x03_P1.27mm_Vertical, F.Cu at (267.1, 46.8)
- added J4: THERM_CONN, Connector_Molex:Molex_Micro-Fit_3.0_43650-0200_1x02_P3.00mm_Horizontal, F.Cu at (99.2, 143.3)
- added L1: 68uH, Inductor_SMD:L_Bourns_SRR1260, F.Cu at (230.1, 68.1)
- added Q1: Q_PMOS_DGS, customFootprints:SISS05DN-T1-GE3, F.Cu at (220.3, 81.4)
- added Q4: Q_PMOS_DGS, customFootprints:SISS05DN-T1-GE3, F.Cu at (210.5, 81.4)
- added R1: 1k, Resistor_SMD:R_0603_1608Metric, F.Cu at (276.4, 48.9)
- added R10: 10, Resistor_SMD:R_0603_1608Metric, F.Cu at (255.0, 75.7)
- added R11: 1k, Resistor_SMD:R_0603_1608Metric, F.Cu at (275.1, 51.4)
- added R12: 1k, Resistor_SMD:R_0603_1608Metric, F.Cu at (247.6, 78.7)
- added R13: 120, Resistor_SMD:R_0603_1608Metric, F.Cu at (255.0, 70.7)
- added R14: 1k, Resistor_SMD:R_0603_1608Metric, F.Cu at (255.0, 73.2)
- added R15: 1k, Resistor_SMD:R_0603_1608Metric, F.Cu at (247.6, 81.2)
- added R16: 1k, Resistor_SMD:R_0603_1608Metric, F.Cu at (259.0, 69.8)
- added R17: 1k, Resistor_SMD:R_0603_1608Metric, F.Cu at (275.6, 59.0)
- added R18: 1k, Resistor_SMD:R_0603_1608Metric, F.Cu at (247.6, 83.7)
- added R19: 3k, Resistor_SMD:R_0603_1608Metric, F.Cu at (271.6, 56.0)
- added R2: 3k, Resistor_SMD:R_0603_1608Metric, F.Cu at (254.7, 68.2)
- added R20: 1k, Resistor_SMD:R_0603_1608Metric, F.Cu at (251.6, 78.2)
- added R21: 10k, Resistor_SMD:R_0603_1608Metric, F.Cu at (271.6, 58.5)
- added R22: 0, Resistor_SMD:R_0603_1608Metric, F.Cu at (268.0, 62.0)
- added R23: 0, Resistor_SMD:R_0603_1608Metric, F.Cu at (275.6, 54.0)
- added R24: 0, Resistor_SMD:R_0603_1608Metric, F.Cu at (259.0, 72.4)
- added R25: 10, Resistor_SMD:R_0603_1608Metric, F.Cu at (275.6, 56.5)
- added R26: 0, Resistor_SMD:R_0603_1608Metric, F.Cu at (264.0, 68.0)
- added R27: 1k, Resistor_SMD:R_0603_1608Metric, F.Cu at (264.0, 65.5)
- added R28: 3k, Resistor_SMD:R_0603_1608Metric, F.Cu at (239.6, 80.7)
- added R29: 1k, Resistor_SMD:R_0603_1608Metric, F.Cu at (263.1, 70.6)
- added R3: 1k, Resistor_SMD:R_0603_1608Metric, F.Cu at (267.6, 57.0)
- added R30: 1, customFootprints:4320_SMD_RES, F.Cu at (218.7, 53.1)
- added R31: 1, customFootprints:4320_SMD_RES, F.Cu at (227.4, 53.1)
- added R32: 1, customFootprints:4320_SMD_RES, F.Cu at (236.2, 53.1)
- added R33: 1, customFootprints:4320_SMD_RES, F.Cu at (218.7, 69.0)
- added R34: 1, customFootprints:4320_SMD_RES, F.Cu at (210.0, 69.0)
- added R35: 1, customFootprints:4320_SMD_RES, F.Cu at (210.0, 53.1)
- added R4: 1k, Resistor_SMD:R_0603_1608Metric, F.Cu at (243.6, 83.1)
- added R5: 1k, Resistor_SMD:R_0603_1608Metric, F.Cu at (268.0, 67.0)
- added R6: 1k, Resistor_SMD:R_0603_1608Metric, F.Cu at (251.6, 83.2)
- added R7: 1k, Resistor_SMD:R_0603_1608Metric, F.Cu at (268.0, 64.5)
- added R8: 270, Resistor_SMD:R_0805_2012Metric, F.Cu at (272.9, 81.0)
- added R9: 30, Resistor_SMD:R_0805_2012Metric, F.Cu at (272.9, 83.9)
- added SW1: RESET, Button_Switch_SMD:SW_SPST_B3U-1000P, F.Cu at (240.1, 71.2)
- added SW2: USER, Button_Switch_SMD:SW_SPST_B3U-1000P, F.Cu at (236.4, 77.3)
- added TP1: ANA_SPARE_1, TestPoint:TestPoint_Pad_D1.0mm, F.Cu at (262.6, 75.8)
- added TP3: PWM_SPARE_1, TestPoint:TestPoint_Pad_D1.0mm, F.Cu at (238.7, 65.6)
- added TP4: PWM_SPARE_2, TestPoint:TestPoint_Pad_D1.0mm, F.Cu at (238.7, 62.6)
- C1: value 22u -> 1u; footprint Capacitor_SMD:C_1210_3225Metric_Pad1.33x2.70mm_HandSolder -> Capacitor_SMD:C_0603_1608Metric
- J1: value Conn_01x02 -> POWER; footprint Connector_PinHeader_2.54mm:PinHeader_1x02_P2.54mm_Vertical_SMD_Pin1Right -> Connector_Molex:Molex_Micro-Fit_3.0_43650-0200_1x02_P3.00mm_Horizontal
- TP2: value TestPoint -> ANA_SPARE_2; footprint TestPoint:TestPoint_Pad_D2.5mm -> TestPoint:TestPoint_Pad_D1.0mm
- U1: value AD820ARMZ -> STM32F103TBU; footprint Package_SO:MSOP-8_3x3mm_P0.65mm -> Package_DFN_QFN:QFN-36-1EP_6x6mm_P0.5mm_EP4.1x4.1mm
- U2: value AD820ARMZ -> MIC5283-3.3ML-TR; footprint Package_SO:MSOP-8_3x3mm_P0.65mm -> Package_DFN_QFN:DFN-8-1EP_3x3mm_P0.65mm_EP1.55x2.4mm
- U4: value Op07DRZ -> TL391B; footprint Package_SO:SOIC-8_3.9x4.9mm_P1.27mm -> Package_TO_SOT_SMD:SOT-23-5
- U5: value ADP1720 -> SN65HVD232; footprint Package_SO:MSOP-8_3x3mm_P0.65mm -> Package_SO:SOIC-8_3.9x4.9mm_P1.27mm
- U6: value TL750L10CD -> MCP1402T-E; footprint Package_SO:SOIC-8_3.9x4.9mm_P1.27mm -> Package_TO_SOT_SMD:SOT-23-5
- moved U6 185.0 mm to (263.1, 59.4), turned to 0 degrees
- moved U5 172.1 mm to (256.5, 60.3), turned to 0 degrees
- moved U4 160.2 mm to (266.4, 53.4)
- moved U2 146.2 mm to (271.7, 47.4)
- moved C1 135.0 mm to (276.4, 46.4)
- moved J1 134.2 mm to (256.6, 55.1), turned to 0 degrees
- moved U3 133.9 mm to (266.5, 82.7)
- moved TP2 101.4 mm to (255.1, 83.5)
- moved U1 100.1 mm to (229.4, 79.3)
Connections:
- C1 pad 1: /powerResistors/IN -> +12V
- J1 pad 1: /PWM_OUT -> Net-(F1-Pad1)
- TP2 pad 1: Net-(D0-Pad1) -> /ANALOG_SPARE_2
- U1 pad 1: (no net) -> +3V3
- U1 pad 2: Net-(C100-Pad1) -> Net-(U1-Pad2)
- U1 pad 3: Net-(R101-Pad2) -> /USER_SW
- U1 pad 4: GND -> /~SW_RESET
- U1 pad 5: (no net) -> GND
- U1 pad 6: Net-(R100-Pad2) -> +3.3VA
- U1 pad 7: +5V -> /THERM_OUTPUT_FILT_AI
- U1 pad 8: (no net) -> /BUCK_OUTPUT_FILT
- U2 pad 1: (no net) -> +12V
- U2 pad 2: Net-(R200-Pad1) -> Net-(U2-Pad2)
- U2 pad 3: Net-(C100-Pad1) -> Net-(U2-Pad3)
- U2 pad 4: GND -> Net-(C2-Pad2)
- U2 pad 5: (no net) -> GND
- U2 pad 6: /PWM_OUT -> +3V3
- U2 pad 7: +12V -> Net-(U2-Pad7)
- U2 pad 8: (no net) -> +3V3
- U3 pad 4: GND -> +3V3
- U3 pad 6: Net-(R200-Pad1) -> Net-(R26-Pad1)
- U3 pad 7: +5V -> GND
- U4 pad 1: (no net) -> Net-(R10-Pad2)
- U4 pad 2: Net-(R400-Pad1) -> GND
- U4 pad 3: Net-(R402-Pad1) -> Net-(D2-Pad1)
- U4 pad 4: GND -> Net-(R5-Pad2)
- U4 pad 5: (no net) -> Net-(C3-Pad2)
- U5 pad 1: GND -> /CAN_UART_P
- U5 pad 2: +12V -> GND
- U5 pad 3: +5V -> +3V3
- U5 pad 4: +12V -> /CAN_UART_N
- U5 pad 5: GND -> Net-(U5-Pad5)
- U5 pad 6: GND -> /CAN_N
- U5 pad 7: GND -> /CAN_P
- U5 pad 8: GND -> Net-(U5-Pad8)
- U6 pad 1: +10V -> GND
- U6 pad 2: GND -> +12V
- U6 pad 3: GND -> /BUCK_PWM
- U6 pad 4: Net-(U6-Pad4) -> GND
Routing:
- net Net-(R402-Pad1): track 97.9 -> 0.00 mm, vias 1 -> 0
- net GND: track 41.6 -> 12.1 mm, vias 45 -> 10
- net /PWM_OUT: track 29.3 -> 0.00 mm
- net Net-(C100-Pad1): track 23.7 -> 0.00 mm
- net Net-(R200-Pad1): track 23.5 -> 0.00 mm
- net Net-(D400-Pad1): track 19.1 -> 0.00 mm
- net Net-(R101-Pad2): track 18.4 -> 0.00 mm
- net Net-(R100-Pad2): track 18.1 -> 0.00 mm
- net Net-(R302-Pad1): track 16.4 -> 0.00 mm
- net +5V: track 14.6 -> 0.00 mm, vias 6 -> 0
- net Net-(R24-Pad2): track 14.2 -> 0.00 mm
- net Net-(R400-Pad1): track 12.7 -> 0.00 mm
- net Net-(R23-Pad1): track 10.1 -> 0.00 mm
- net +12V: track 8.11 -> 0.00 mm, vias 12 -> 0
- net +10V: track 7.38 -> 0.00 mm
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- removed copper zone on F.Cu, net +12V
- removed copper zone on F.Cu, net /powerResistors/IN
- removed copper zone on F.Cu, net Net-(D0-Pad1)

Commit message: Preliminary Layout Complete
Parts:
- removed the C2 at (178.3, 94.0)
- removed the C3 at (145.8, 94.0)
- removed the C3 at (251.0, 75.3)
- removed the C4 at (112.3, 94.0)
- removed the C5 at (101.1, 44.2)
- removed the C6 at (134.6, 44.2)
- removed the C7 at (167.1, 44.2)
- removed R0: 1, customFootprints:4320_SMD_RES
- removed the R1 at (140.2, 100.6)
- removed the R2 at (106.7, 100.6)
- removed the R3 at (106.7, 50.8)
- removed the R4 at (140.2, 50.8)
- removed the R5 at (172.7, 50.8)
- removed the TP1 at (183.4, 131.1)
- added C3: 0.1u, Capacitor_SMD:C_0603_1608Metric, F.Cu at (112.5, 154.4)
- moved R23 188.1 mm to (105.7, 134.6), turned to 180 degrees
- moved R19 187.0 mm to (103.1, 137.2), turned to 90 degrees
- moved R21 184.5 mm to (103.1, 133.8), turned to 270 degrees
- moved R7 181.4 mm to (110.5, 154.4), turned to 270 degrees
- moved U4 181.2 mm to (115.6, 154.0), turned to 90 degrees
- moved C1 179.4 mm to (122.2, 138.2)
- moved R17 179.2 mm to (122.2, 151.6), turned to 270 degrees
- moved R22 178.7 mm to (105.7, 136.7), turned to 180 degrees
- moved J1 176.9 mm to (105.1, 146.6), turned to 180 degrees
- moved U2 175.6 mm to (122.9, 140.7)
- moved R5 175.5 mm to (113.5, 150.4)
- moved R3 172.8 mm to (117.9, 143.3)
- moved C13 172.5 mm to (132.6, 153.9), turned to 90 degrees
- moved C20 170.4 mm to (116.8, 131.8), turned to 270 degrees
- moved R1 169.7 mm to (134.1, 141.5), turned to 90 degrees
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Routing:
- net Net-(C5-Pad1): track 55.6 -> 0.00 mm
- net Net-(R32-Pad2): track 0.00 -> 49.3 mm
- net /powerResistors/IN: track 40.5 -> 0.00 mm
- net Net-(C16-Pad2): track 0.00 -> 34.8 mm
- net Net-(C4-Pad1): track 28.3 -> 0.00 mm
- net Net-(C6-Pad1): track 28.3 -> 0.00 mm
- net Net-(C3-Pad1): track 27.3 -> 0.00 mm
- net Net-(C7-Pad1): track 27.3 -> 0.00 mm
- net Net-(R32-Pad1): track 0.00 -> 23.9 mm
- net Net-(R31-Pad2): track 0.00 -> 23.6 mm
- net Net-(R30-Pad2): track 0.00 -> 20.5 mm
- net Net-(R34-Pad2): track 0.00 -> 20.4 mm
- net GND: track 12.1 -> 2.03 mm, vias 10 -> 4
Other:
- outline, holes or cut-outs redrawn

Commit message: Finished Layout
Parts:
- removed TH400: Thermistor, Resistor_THT:R_Axial_DIN0204_L3.6mm_D1.6mm_P2.54mm_Vertical
- moved G*** 75.8 mm to (131.3, 117.1)
- moved G*** 75.8 mm to (150.4, 118.1)
- moved Q4 41.4 mm to (165.6, 136.1)
- moved R25 40.9 mm to (168.7, 138.4), turned to 90 degrees
- moved C15 40.8 mm to (164.3, 132.6)
- moved R20 38.3 mm to (168.7, 141.5)
- moved U6 37.8 mm to (165.6, 140.5)
- moved C18 37.6 mm to (162.6, 139.7)
- moved D6 36.6 mm to (167.9, 131.4), turned to 90 degrees
- moved L1 32.5 mm to (176.3, 136.1)
- moved C16 31.6 mm to (183.6, 140.2)
- moved R28 31.6 mm to (186.7, 140.2)
- moved R29 31.6 mm to (186.7, 143.8)
- moved R18 16.7 mm to (141.7, 148.1), turned to 90 degrees
- moved J2 11.4 mm to (170.7, 147.1)
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Routing:
- net /BUCK_OUTPUT_AI: track 0.00 -> 78.9 mm, vias 0 -> 2
- net GND: track 2.03 -> 51.6 mm, vias 4 -> 48
- net /~SW_RESET: track 0.00 -> 32.3 mm, vias 0 -> 2
- net /BUCK_PWM: track 0.00 -> 28.7 mm, vias 0 -> 2
- net /THERM_OUTPUT_FILT_AI: track 0.00 -> 22.9 mm, vias 0 -> 2
- net /USER_SW: track 0.00 -> 20.5 mm, vias 0 -> 2
- net +3V3: track 0.00 -> 18.2 mm, vias 0 -> 12
- net /CAN_P: track 0.00 -> 16.7 mm
- net /CAN_N: track 0.00 -> 16.1 mm
- net /BATT_VOLTAGE_AI: track 0.00 -> 15.3 mm
- net /CAN_UART_N: track 0.00 -> 14.7 mm
- net /CAN_UART_P: track 0.00 -> 14.7 mm
- net Net-(D2-Pad1): track 0.00 -> 14.1 mm
- net Net-(R26-Pad1): track 0.00 -> 13.2 mm
- net Net-(R10-Pad2): track 0.00 -> 13.0 mm
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- added copper zone on F.Cu, net +12V
- added copper zone on F.Cu, net +3V3
- added copper zone on In2.Cu, net +3V3
- added copper zone on F.Cu, net Net-(C16-Pad2)
- added copper zone on F.Cu, net Net-(C3-Pad2)
- added copper zone on F.Cu, net Net-(D6-Pad1)
- added copper zone on F.Cu, net Net-(F1-Pad1)
- added copper zone on F.Cu, net Net-(J4-Pad1)
- removed copper zone on In2.Cu, net +5V
Other:
- outline, holes or cut-outs redrawn
- board text added: "2022"
- board text added: "Designed by: Walsh Bros Inc."
- board text removed: "2021"
- board text removed: "Designed by: Daniel Walsh"

Commit message: Adjusted Silk Screen
Changed lines of the file:
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@@
     (tags "SOIC SO")
     (attr smd)
-    (fp_text reference U3 (at 8.128 -1.524) (layer F.SilkS)
+    (fp_text reference U3 (at 1.27 3.556) (layer F.SilkS)
       (effects (font (size 1 1) (thickness 0.15)))
     )
@@
     (tags resistor)
     (attr smd)
-    (fp_text reference R8 (at 0.1505 -1.778 90) (layer F.SilkS)
+    (fp_text reference R8 (at -0.1035 -1.778 90) (layer F.SilkS)
       (effects (font (size 1 1) (thickness 0.15)))
     )
@@
     (tags capacitor)
     (attr smd)
-    (fp_text reference C4 (at -1.27 -1.778 90) (layer F.SilkS)
+    (fp_text reference C4 (at 3.302 0 90) (layer F.SilkS)
       (effects (font (size 1 1) (thickness 0.15)))
     )
@@
     (tags capacitor)
     (attr smd)
-    (fp_text reference C5 (at -2.54 0) (layer F.SilkS)
+    (fp_text reference C5 (at -0.013 -1.524) (layer F.SilkS)
       (effects (font (size 1 1) (thickness 0.15)))
     )
@@
     (tags capacitor)
     (attr smd)
-    (fp_text reference C6 (at 0.241 -1.524 90) (layer F.SilkS)
+    (fp_text reference C6 (at 2.54 0 90) (layer F.SilkS)
       (effects (font (size 1 1) (thickness 0.15)))
     )
@@
     (tags capacitor)
     (attr smd)
-    (fp_text reference C7 (at -0.013 3.302) (layer F.SilkS)
+    (fp_text reference C7 (at 2.807 0) (layer F.SilkS)
       (effects (font (size 1 1) (thickness 0.15)))
     )
@@
     (tags capacitor)
     (attr smd)
-    (fp_text reference C8 (at -2.54 0.254 90) (layer F.SilkS)
+    (fp_text reference C8 (at -2.54 0 90) (layer F.SilkS)
       (effects (font (size 1 1) (thickness 0.15)))
     )
@@
     (tags capacitor)
     (attr smd)
-    (fp_text reference C15 (at 3.061 0 90) (layer F.SilkS)
+    (fp_text reference C15 (at -0.241 -1.524 90) (layer F.SilkS)
       (effects (font (size 1 1) (thickness 0.15)))
     )
@@
     (tags capacitor)
     (attr smd)
-    (fp_text reference C18 (at -3.048 0 90) (layer F.SilkS)
+    (fp_text reference C18 (at 0.254 1.524 90) (layer F.SilkS)
       (effects (font (size 1 1) (thickness 0.15)))
     )
@@
     (tags LED)
     (attr smd)
-    (fp_text reference D3 (at -2.3115 -3.81 90) (layer F.SilkS)
+    (fp_text reference D3 (at 0.7365 1.778 90) (layer F.SilkS)
       (effects (font (size 1 1) (thickness 0.15)))
     )
@@
     (tags LED)
     (attr smd)
-    (fp_text reference D4 (at -2.286 -3.81 90) (layer F.SilkS)
+    (fp_text reference D4 (at 0.762 -1.524 90) (layer F.SilkS)
       (effects (font (size 1 1) (thickness 0.15)))
     )
@@
     (tags inductor)
     (attr smd)
-    (fp_text reference FB1 (at 0 1.524) (layer F.SilkS)
+    (fp_text reference FB1 (at -1.27 -1.524) (layer F.SilkS)
       (effects (font (size 1 1) (thickness 0.15)))
     )
@@
   (module customFootprints:SISS05DN-T1-GE3 (layer F.Cu)
     (at 115.824 139.192)
-    (fp_text reference Q1 (at -4.064 0 90) (layer F.SilkS)
+    (fp_text reference Q1 (at -2.54 0 90) (layer F.SilkS)
       (effects (font (size 1 1) (thickness 0.15)))
     )
-    (fp_text value Q_PMOS_DGS (at -2.54 1.524 90) (layer F.SilkS)
+    (fp_text value Q_PMOS_DGS (at -2.54 1.524 90) (layer F.SilkS) hide
       (effects (font (size 1 1) (thickness 0.15)))
     )
@@
   (module customFootprints:SISS05DN-T1-GE3 (layer F.Cu)
     (at 165.608 136.144 90)
-    (fp_text reference Q4 (at 2.794 -0.254 180) (layer F.SilkS)
+    (fp_text reference Q4 (at 2.794 0.254 180) (layer F.SilkS)
       (effects (font (size 1 1) (thickness 0.15)))
     )
-    (fp_text value Q_PMOS_DGS (at 6.35 -5.842) (layer F.SilkS)
+    (fp_text value Q_PMOS_DGS (at 6.35 -5.842) (layer F.SilkS) hide
       (effects (font (size 1 1) (thickness 0.15)))
     )
@@
     (tags resistor)
     (attr smd)
-    (fp_text reference R18 (at 0 3.302 90) (layer F.SilkS)
+    (fp_text reference R18 (at 2.857 0 90) (layer F.SilkS)
       (effects (font (size 1 1) (thickness 0.15)))
     )
@@
     (tags resistor)
     (attr smd)
-    (fp_text reference R20 (at -3.111 0 90) (layer F.SilkS)
+    (fp_text reference R20 (at -2.223 -1.524 270) (layer F.SilkS)
       (effects (font (size 1 1) (thickness 0.15)))
     )
@@
     (tags resistor)
     (attr smd)
-    (fp_text reference R27 (at 2.985 0.254) (layer F.SilkS)
+    (fp_text reference R27 (at 0 -1.524) (layer F.SilkS)
       (effects (font (size 1 1) (thickness 0.15)))
     )
@@
   (module customFootprints:4320_SMD_RES (layer F.Cu)
     (at 172.72 100.584 270)
-    (fp_text reference R30 (at 0 11.43 90) (layer F.SilkS)
+    (fp_text reference R30 (at 0 8.382 90) (layer F.SilkS)
       (effects (font (size 1 1) (thickness 0.15)))
     )
@@
   (module customFootprints:4320_SMD_RES (layer F.Cu)
     (at 140.716 100.584 270)
-    (fp_text reference R31 (at 0 11.43 90) (layer F.SilkS)
+    (fp_text reference R31 (at 0 8.128 90) (layer F.SilkS)
       (effects (font (size 1 1) (thickness 0.15)))
     )
@@
   (module customFootprints:4320_SMD_RES (layer F.Cu)
     (at 106.68 50.8 270)
-    (fp_text reference R32 (at 0 11.43 90) (layer F.SilkS)
+    (fp_text reference R32 (at 0 -8.382 90) (layer F.SilkS)
       (effects (font (size 1 1) (thickness 0.15)))
     )
@@
   (module customFootprints:4320_SMD_RES (layer F.Cu)
     (at 106.68 100.584 90)
-    (fp_text reference R33 (at 0 11.43 90) (layer F.SilkS)
+    (fp_text reference R33 (at 0 -8.128 90) (layer F.SilkS)
       (effects (font (size 1 1) (thickness 0.15)))
     )
@@
   (module customFootprints:4320_SMD_RES (layer F.Cu)
     (at 140.208 50.8 90)
-    (fp_text reference R34 (at 0 11.43 90) (layer F.SilkS)
+    (fp_text reference R34 (at 0 8.382 90) (layer F.SilkS)
       (effects (font (size 1 1) (thickness 0.15)))
     )
@@
   (module customFootprints:4320_SMD_RES (layer F.Cu)
     (at 172.212 50.8 90)
-    (fp_text reference R35 (at 0 11.43 90) (layer F.SilkS)
+    (fp_text reference R35 (at 0 8.382 90) (layer F.SilkS)
       (effects (font (size 1 1) (thickness 0.15)))
     )

Commit message: small ss and copper changes
Parts:
- added C21: 1u, Capacitor_SMD:C_0603_1608Metric, F.Cu at (164.0, 131.7)
- added C22: 1u, Capacitor_SMD:C_0603_1608Metric, F.Cu at (182.9, 128.7)
- added C23: 1u, Capacitor_SMD:C_0603_1608Metric, F.Cu at (185.2, 140.2)
- added G***: LOGO, customFootprints:woodStove_logo, F.Cu at (141.0, 75.4)
- 12V POWER: renamed from J1
- CAN CONN: renamed from J2
- moved 12V POWER 1.36 mm to (105.1, 147.9)
- moved THERMISTOR 0.92 mm to (98.7, 136.0)
- moved CAN CONN 0.80 mm to (170.7, 147.9)
- moved C15 0.74 mm to (164.0, 133.2), turned to 0 degrees
- renumbered SW1 to RESET, J3 to SWD, J4 to THERMISTOR, SW2 to USER
Connections:
- U1 pad 12: Net-(U1-Pad12) -> /THERM_OUTPUT_UNFILT_AI
Routing:
- net /THERM_OUTPUT_UNFILT_AI: track 0.00 -> 36.2 mm, vias 0 -> 2
- net /BUCK_OUTPUT_AI: track 78.9 -> 74.3 mm
- net /CAN_N: track 16.1 -> 14.6 mm
- net /CAN_P: track 16.7 -> 15.3 mm
- net +12V: track 10.2 -> 8.96 mm, vias 7 -> 6
- net GND: track 51.6 -> 52.3 mm, vias 48 -> 50
- net /USER_SW: track 20.5 -> 21.2 mm
- net +3V3: vias 12 -> 13
Other:
- net class CAN added: clearance 0.2, trace_width 0.127, via_dia 0.8, via_drill 0.4
- rule trace_min: 0.2 -> 0.127
- board text added: "Designed by: Walsh^2 Inc."
- board text added: "Jan. 2022"
- board text removed: "2022"
- board text removed: "Designed by: Walsh Bros Inc."

Commit message: Hopefully the ordered gerbers
Parts:
- C20, R27: moved to B.Cu
- POWER (12V): renamed from 12V POWER
- moved C20 14.3 mm to (128.0, 141.3), turned to 270 degrees
- moved R27 14.1 mm to (129.6, 141.3), turned to 90 degrees
- moved C19 8.47 mm to (117.9, 131.3)
Connections:
- U3 pad 4: +3V3 -> GND
- U3 pad 7: GND -> +3V3
Routing:
- net Net-(R26-Pad1): track 13.2 -> 30.5 mm, vias 0 -> 1
- net /THERM_OUTPUT_FILT_AI: track 22.9 -> 10.4 mm, vias 2 -> 1
- net /THERM_OUTPUT_UNFILT_AI: track 36.2 -> 40.4 mm
- net /BUCK_OUTPUT_AI: track 74.3 -> 78.4 mm
- net +3V3: track 18.2 -> 19.0 mm
- net GND: track 52.3 -> 51.8 mm, vias 50 -> 51
